File: STM32/STM32.kicad_sch (KiCad schematic)
At the start: 24 parts, among them J1 USB_B_Micro, J2 Conn_01x04_Pin, SW1 SW_SPDT, U1 STM32F103C8Tx, U2 AMS1117-3.3, Y1 Crystal_GND24

Commit message: Push to PC
Push to PC
Parts:
- added U3: TMP112BIDRLT, TMP112:DRL0006A, symbol TMP1112:TMP112BIDRLT
Connections:
- net +3.3V: now also U3.5 (V+)
- net GND: now also U1.23 (VSS), U1.35 (VSS), U1.47 (VSS), U1.8 (VSSA), U3.2 (GND), U3.3 (ALERT), U3.4 (ADD0)
- net I2C2_SCL: now reaches U1.21 (PB10)
- net I2C2_SCL: now also U3.1 (SCL)
- net I2C2SDA: now reaches U1.22 (PB11)
- net I2C2SDA: now also U3.6 (SDA)
Other:
- note added: "Address: 40h"
- moved on the sheet: C1, C10, C11, C2, C3, C4, C5, C6, C7, C8, C9, FB1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

Commit message: Push to save
Parts:
- added U4: TMAG5170A1QDGKR, DGK0008A-IPC_A, symbol EMI Sensor:TMAG5170A1QDGKR
Connections:
- net I2C2SDA renamed I2C2_SDA
Other:
- moved on the sheet: C1, C10, C11, C2, C3, C4, C5, C6, C7, C8, C9, FB1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
